File: hardware/star/star.sch (EAGLE design)
At the start: 157 parts, among them IC1 MAX481CSA, IC2 LD117AS12TR, IC22 LD117AS12TR, IC3 74HCT08D, IC4 7404D, IC5 LM317MABDT, IC6 LM317MABDT, IC7 LM317MABDT, K1 T90-12VDC-TL-A, K2 T90-12VDC-TL-A, Q1 35A/25V/8.5mΩ, Q2 35A/25V/8.5mΩ, Q3 35A/25V/8.5mΩ, Q4 35A/25V/8.5mΩ, T1 T_PNP_MMBT5401_CHANGJ_SOT23-B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, T2 T_PNP_MMBT5401_CHANGJ_SOT23-B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, T3 T_PNP_MMBT5401_CHANGJ_SOT23-B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, T4 T_PNP_MMBT5401_CHANGJ_SOT23-B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, U1 TCLT1600, X1 MKDSN1,5/2-5,08, X3 MKDSN1,5/5-5,08

Commit message: manual traces
Parts:
- added C33: 1uf, rcl:C-USC0805
- added IC8: MAX481CSA, maxim:MAX481CSA
- added P1: B3B-PH-K, con-jst-ph:B3B-PH-K
- added R5: 120, rcl:R-US_R0603
Connections:
- new net N$5: IC8G$1.B, P1.2, R5.2
- new net N$6: IC8G$1.A, P1.3, R5.1
- net +3V3: now also C33.1, IC8P.VCC
- net 2: now also IC8G$1.RO
- net 4: now also IC8G$1.DI
- net A4: now also IC8G$1.DE
- net A5: now also IC8G$1.RE/
- net GND: now also C33.2, IC8P.GND, P1.1
Other:
- note added: "2nd RS485 (DMX512)"
Changed lines of the file:
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@@
 <setting verticaltext="up"/>
 </settings>
-<grid distance="0.1" unitdist="inch" unit="inch" style="lines" multiple="1" display="no" altdistance="0.01" altunitdist="inch" altunit="inch"/>
+<grid distance="0.1" unitdist="inch" unit="inch" style="lines" multiple="1" display="yes" altdistance="0.01" altunitdist="inch" altunit="inch"/>
 <layers>
 <layer number="1" name="Top" color="4" fill="1" visible="no" active="no"/>
@@
 <part name="P+15" library="supply1" library_urn="urn:adsk.eagle:library:371" deviceset="+5V" device=""/>
 <part name="P+25" library="supply1" library_urn="urn:adsk.eagle:library:371" deviceset="+5V" device=""/>
+<part name="IC8" library="maxim" library_urn="urn:adsk.eagle:library:269" deviceset="MAX481CSA" device="" package3d_urn="urn:adsk.eagle:package:17511/1">
+<attribute name="LCSC_PART" value="C8963"/>
+</part>
+<part name="GND29" library="supply1" library_urn="urn:adsk.eagle:library:371" deviceset="GND" device=""/>
+<part name="+3V7" library="supply1" library_urn="urn:adsk.eagle:library:371" deviceset="+3V3" device=""/>
+<part name="C33" library="rcl" library_urn="urn:adsk.eagle:library:334" deviceset="C-US" device="C0805" package3d_urn="urn:adsk.eagle:package:23617/2" value="1uf">
+<spice>
+<pinmapping spiceprefix="C">
+<pinmap gate="G$1" pin="1" pinorder="1"/>
+<pinmap gate="G$1" pin="2" pinorder="2"/>
+</pinmapping>
+</spice>
+<attribute name="LCSC_PART" value="C15849"/>
+</part>
+<part name="R5" library="rcl" library_urn="urn:adsk.eagle:library:334" deviceset="R-US_" device="R0603" package3d_urn="urn:adsk.eagle:package:23555/3" value="120">
+<spice>
+<pinmapping spiceprefix="R">
+<pinmap gate="G$1" pin="1" pinorder="1"/>
+<pinmap gate="G$1" pin="2" pinorder="2"/>
+</pinmapping>
+</spice>
+<attribute name="LCSC_PART" value="C22787"/>
+</part>
+<part name="P1" library="con-jst-ph" library_urn="urn:adsk.eagle:library:37597460" deviceset="B3B-PH-K" device="" package3d_urn="urn:adsk.eagle:package:37597508/1"/>
+<part name="GND30" library="supply1" library_urn="urn:adsk.eagle:library:371" deviceset="GND" device=""/>
 </parts>
 <sheets>
@@
 <text x="401.32" y="279.4" size="1.778" layer="98">5v Controlled Output
 (aka Lasers)</text>
+<wire x1="231.14" y1="147.32" x2="314.96" y2="147.32" width="0.2032" layer="98"/>
+<wire x1="314.96" y1="147.32" x2="314.96" y2="81.28" width="0.254" layer="98"/>
+<wire x1="314.96" y1="81.28" x2="231.14" y2="81.28" width="0.254" layer="98"/>
+<wire x1="231.14" y1="81.28" x2="231.14" y2="147.32" width="0.254" layer="98"/>
+<text x="236.22" y="139.7" size="2.54" layer="98">2nd RS485
+(DMX512)</text>
 </plain>
 <instances>
@@
 <attribute name="VALUE" x="78.74" y="403.86" size="1.778" layer="96" rot="R90"/>
 </instance>
+<instance part="IC8" gate="G$1" x="274.32" y="109.22" smashed="yes" rot="R180">
+<attribute name="NAME" x="284.48" y="95.25" size="1.778" layer="95" rot="R180"/>
+<attribute name="VALUE" x="284.48" y="124.46" size="1.778" layer="96" rot="R180"/>
+<attribute name="LCSC_PART" x="274.32" y="109.22" size="1.778" layer="96" rot="R180" display="off"/>
+</instance>
+<instance part="IC8" gate="P" x="299.72" y="109.22" smashed="yes" rot="R180">
+<attribute name="NAME" x="300.482" y="109.982" size="1.778" layer="95" rot="R180"/>
+</instance>
+<instance part="GND29" gate="1" x="299.72" y="121.92" smashed="yes" rot="R180">
+<attribute name="VALUE" x="302.26" y="124.46" size="1.778" layer="96" rot="R180"/>
+</instance>
+<instance part="+3V7" gate="G$1" x="299.72" y="96.52" smashed="yes" rot="R180">
+<attribute name="VALUE" x="302.26" y="101.6" size="1.778" layer="96" rot="R270"/>
+</instance>
+<instance part="C33" gate="G$1" x="309.88" y="104.14" smashed="yes" rot="R180">
+<attribute name="NAME" x="308.864" y="103.505" size="1.778" layer="95" rot="R180"/>
+<attribute name="VALUE" x="308.864" y="108.331" size="1.778" layer="96" rot="R180"/>
+<attribute name="LCSC_PART" x="309.88" y="104.14" size="1.778" layer="96" rot="R180" display="off"/>
+</instance>
+<instance part="R5" gate="G$1" x="254" y="106.68" smashed="yes" rot="R270">
+<attribute name="NAME" x="255.4986" y="110.49" size="1.778" layer="95" rot="R270"/>
+<attribute name="VALUE" x="250.698" y="110.49" size="1.778" layer="96" rot="R270"/>
+<attribute name="LCSC_PART" x="254" y="106.68" size="1.778" layer="96" rot="R270" display="off"/>
+</instance>
+<instance part="P1" gate="G$1" x="243.84" y="96.52" smashed="yes" rot="R180">
+<attribute name="NAME" x="245.11" y="90.805" size="1.778" layer="95" rot="R180"/>
+<attribute name="VALUE" x="245.11" y="104.14" size="1.778" layer="95" rot="R180"/>
+</instance>
+<instance part="GND30" gate="1" x="251.46" y="88.9" smashed="yes">
+<attribute name="VALUE" x="248.92" y="86.36" size="1.778" layer="96"/>
+</instance>
 </instances>
 <busses>
@@
 <label x="337.82" y="332.74" size="1.778" layer="95" rot="R90"/>
 </segment>
+<segment>
+<wire x1="294.64" y1="96.52" x2="287.02" y2="96.52" width="0.762" layer="92"/>
+<label x="297.18" y="93.98" size="1.778" layer="96" rot="R180"/>
+</segment>
 </bus>
 <bus name="NEBULA:A[0..15]">
@@
 <label x="337.82" y="312.42" size="1.778" layer="95" rot="R90"/>
 </segment>
+<segment>
+<wire x1="294.64" y1="132.08" x2="287.02" y2="132.08" width="0.762" layer="92"/>
+<label x="289.56" y="134.62" size="1.778" layer="95"/>
+</segment>
 </bus>
 <bus name="EXP_ULN:EXP_ULN[0..7]">
@@
 <junction x="248.92" y="241.3"/>
 </segment>
+<segment>
+<pinref part="GND29" gate="1" pin="GND"/>
+<pinref part="IC8" gate="P" pin="GND"/>
+<wire x1="299.72" y1="116.84" x2="299.72" y2="119.38" width="0.1524" layer="91"/>
+<pinref part="C33" gate="G$1" pin="2"/>
+<wire x1="309.88" y1="119.38" x2="309.88" y2="109.22" width="0.1524" layer="91"/>
+<wire x1="299.72" y1="119.38" x2="309.88" y2="119.38" width="0.1524" layer="91"/>
+<junction x="299.72" y="119.38"/>
+</segment>
+<segment>
+<pinref part="P1" gate="G$1" pin="1"/>
+<pinref part="GND30" gate="1" pin="GND"/>
+<wire x1="248.92" y1="93.98" x2="251.46" y2="93.98" width="0.1524" layer="91"/>
+<wire x1="251.46" y1="93.98" x2="251.46" y2="91.44" width="0.1524" layer="91"/>
+</segment>
 </net>
 <net name="N$1" class="0">
@@
 <wire x1="96.52" y1="325.12" x2="96.52" y2="327.66" width="0.1524" layer="91"/>
 </segment>
+<segment>
+<pinref part="IC8" gate="P" pin="VCC"/>
+<pinref part="+3V7" gate="G$1" pin="+3V3"/>
+<wire x1="299.72" y1="99.06" x2="299.72" y2="101.6" width="0.1524" layer="91"/>
+<pinref part="C33" gate="G$1" pin="1"/>
+<wire x1="309.88" y1="101.6" x2="309.88" y2="99.06" width="0.1524" layer="91"/>
+<wire x1="309.88" y1="99.06" x2="299.72" y2="99.06" width="0.1524" layer="91"/>
+<junction x="299.72" y="99.06"/>
+</segment>
 </net>
 <net name="36" class="0">
@@
 <wire x1="58.42" y1="355.6" x2="60.96" y2="355.6" width="0.1524" layer="91"/>
 <wire x1="60.96" y1="355.6" x2="60.96" y2="335.28" width="0.1524" layer="91"/>
+<label x="60.96" y="342.9" size="1.778" layer="95"/>
 </segment>
 </net>
@@
 <pinref part="IC1" gate="G$1" pin="RO"/>
 <wire x1="58.42" y1="340.36" x2="58.42" y2="335.28" width="0.1524" layer="91"/>
+<label x="58.42" y="337.82" size="1.778" layer="95"/>
 </segment>
 </net>
@@
 <label x="210.82" y="335.28" size="1.778" layer="95"/>
 </segment>
+<segment>
+<pinref part="IC8" gate="G$1" pin="DI"/>
+<wire x1="287.02" y1="116.84" x2="289.56" y2="116.84" width="0.1524" layer="91"/>
+<wire x1="289.56" y1="116.84" x2="289.56" y2="96.52" width="0.1524" layer="91"/>
+<label x="289.56" y="101.6" size="1.778" layer="95"/>
+</segment>
 </net>
 <net name="2" class="0">
@@
 <label x="210.82" y="332.74" size="1.778" layer="95"/>
 </segment>
+<segment>
+<pinref part="IC8" gate="G$1" pin="RO"/>
+<wire x1="287.02" y1="101.6" x2="287.02" y2="96.52" width="0.1524" layer="91"/>
+<label x="287.02" y="99.06" size="1.778" layer="95"/>
+</segment>
 </net>
 <net name="15" class="0">
@@
 <label x="314.96" y="335.28" size="1.778" layer="95"/>
 </segment>
+<segment>
+<pinref part="IC8" gate="G$1" pin="DE"/>
+<wire x1="287.02" y1="111.76" x2="292.1" y2="111.76" width="0.1524" layer="91"/>
+<wire x1="292.1" y1="111.76" x2="292.1" y2="132.08" width="0.1524" layer="91"/>
+<label x="289.56" y="129.54" size="1.778" layer="95"/>
+</segment>
 </net>
 <net name="A5" class="0">
@@
 <label x="314.96" y="332.74" size="1.778" layer="95"/>
 </segment>
+<segment>
+<pinref part="IC8" gate="G$1" pin="RE/"/>
+<wire x1="287.02" y1="106.68" x2="294.64" y2="106.68" width="0.1524" layer="91"/>
+<wire x1="294.64" y1="106.68" x2="294.64" y2="132.08" width="0.1524" layer="91"/>
+<label x="294.64" y="127" size="1.778" layer="95"/>
+</segment>
 </net>
 <net name="A6" class="0">
@@
 </segment>
 </net>
+<net name="N$5" class="0">
+<segment>
+<pinref part="IC8" gate="G$1" pin="B"/>
+<pinref part="R5" gate="G$1" pin="2"/>
+<wire x1="261.62" y1="96.52" x2="261.62" y2="101.6" width="0.1524" layer="91"/>
+<wire x1="261.62" y1="101.6" x2="261.62" y2="106.68" width="0.1524" layer="91"/>
+<wire x1="254" y1="101.6" x2="261.62" y2="101.6" width="0.1524" layer="91"/>
+<junction x="261.62" y="101.6"/>
+<pinref part="P1" gate="G$1" pin="2"/>
+<wire x1="248.92" y1="96.52" x2="261.62" y2="96.52" width="0.1524" layer="91"/>
+</segment>
+</net>
+<net name="N$6" class="0">
+<segment>
+<pinref part="IC8" gate="G$1" pin="A"/>
+<wire x1="259.08" y1="99.06" x2="259.08" y2="111.76" width="0.1524" layer="91"/>
+<wire x1="259.08" y1="111.76" x2="261.62" y2="111.76" width="0.1524" layer="91"/>
+<pinref part="R5" gate="G$1" pin="1"/>
+<wire x1="254" y1="111.76" x2="259.08" y2="111.76" width="0.1524" layer="91"/>
+<junction x="259.08" y="111.76"/>
+<pinref part="P1" gate="G$1" pin="3"/>
+<wire x1="248.92" y1="99.06" x2="259.08" y2="99.06" width="0.1524" layer="91"/>
+</segment>
+</net>

Commit message: critical traces routed
Parts:
- added C34: 1uf, rcl:C-USC0805
- added C37: 10uf, rcl:C-USC0603
- added IC9: LD117AS12TR, v-reg:LD117AS12TR
- added JP2: (no value), pinhead:PINHD-2X2
Connections:
- net +12V: now also C34.1, IC9.IN
- net +5V: now also C37.1, IC9.OUT
- net GND: now also C34.2, C37.2, IC9.ADJ, JP2.1, JP2.2, JP2.3, JP2.4
Other:
- note added: "Holes & Ground"
- note removed: "Holes"
- moved on the sheet: 5V_CTRL_LAZERS, C10, C11, C12, C2, C24, C25, C26, C27, C28, C29, C30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

Commit message: update
Parts:
- added R6: R_0R_1206, JLC PCB Basic Parts_loc:R_0R_1206
- FIRE: device con-phoenix-508:MKDSN1,5/8-5,08 -> con-phoenix-508-jm:MKDSN1,5/8-5,08
- POWER_IN: device con-phoenix-508:MKDSN1,5/4-5,08 -> con-phoenix-508-jm:MKDSN1,5/4-5,08
- R132: value 12k -> 1k; LCSC_PART C22790 -> C21190
- X1: device con-phoenix-508:MKDSN1,5/2-5,08 -> con-phoenix-508-jm:MKDSN1,5/2-5,08
- X3: device con-phoenix-508:MKDSN1,5/5-5,08 -> con-phoenix-508-jm:MKDSN1,5/5-5,08
Connections:
- net GND: now also R6.1
- net GND2: now also R6.2
Changed lines of the file:
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@@
 <setting verticaltext="up"/>
 </settings>
-<grid distance="0.1" unitdist="inch" unit="inch" style="lines" multiple="1" display="yes" altdistance="0.01" altunitdist="inch" altunit="inch"/>
+<grid distance="0.1" unitdist="inch" unit="inch" style="lines" multiple="1" display="no" altdistance="0.01" altunitdist="inch" altunit="inch"/>
 <layers>
 <layer number="1" name="Top" color="4" fill="1" visible="no" active="no"/>
@@
 </part>
 <part name="GND1" library="supply1" library_urn="urn:adsk.eagle:library:371" deviceset="GND" device=""/>
-<part name="POWER_IN" library="con-phoenix-508" library_urn="urn:adsk.eagle:library:176" deviceset="MKDSN1,5/4-5,08" device="" package3d_urn="urn:adsk.eagle:package:9636/1"/>
+<part name="POWER_IN" library="con-phoenix-508-jm" deviceset="MKDSN1,5/4-5,08" device="" package3d_urn="urn:adsk.eagle:package:9636/1"/>
 <part name="+3V4" library="supply1" library_urn="urn:adsk.eagle:library:371" deviceset="+3V3" device=""/>
 <part name="NEBULA_A" library="MCP23017-E_SO" library_urn="urn:adsk.eagle:library:37530508" deviceset="MCP23017-E/SO" device="" package3d_urn="urn:adsk.eagle:package:37530511/1">
@@
 <part name="JTAG" library="pinhead" library_urn="urn:adsk.eagle:library:325" deviceset="PINHD-1X5" device="" package3d_urn="urn:adsk.eagle:package:22469/2"/>
 <part name="GND47" library="supply1" library_urn="urn:adsk.eagle:library:371" deviceset="GND" device=""/>
-<part name="STAR_INPUT" library="con-jst-ph" library_urn="urn:adsk.eagle:library:37597460" deviceset="B8B-PH-K" device="" package3d_urn="urn:adsk.eagle:package:37597503/1"/>
+<part name="STAR_INPUT" library="con-jst-ph" library_urn="urn:adsk.eagle:library:37597460" deviceset="B8B-PH-K" device="" package3d_urn="urn:adsk.eagle:package:37597503/2"/>
 <part name="IC1" library="maxim" library_urn="urn:adsk.eagle:library:269" deviceset="MAX481CSA" device="" package3d_urn="urn:adsk.eagle:package:17511/1">
 <attribute name="LCSC_PART" value="C8963"/>
@@
 <attribute name="LCSC_PART" value="C4190"/>
 </part>
-<part name="R132" library="rcl" library_urn="urn:adsk.eagle:library:334" deviceset="R-US_" device="R0603" package3d_urn="urn:adsk.eagle:package:23555/3" value="12k">
+<part name="R132" library="rcl" library_urn="urn:adsk.eagle:library:334" deviceset="R-US_" device="R0603" package3d_urn="urn:adsk.eagle:package:23555/3" value="1k">
 <spice>
 <pinmapping spiceprefix="R">
@@
 </pinmapping>
 </spice>
-<attribute name="LCSC_PART" value="C22790"/>
+<attribute name="LCSC_PART" value="C21190"/>
 </part>
 <part name="GND99" library="supply1" library_urn="urn:adsk.eagle:library:371" deviceset="GND" device=""/>
@@
 <part name="+3V52" library="supply1" library_urn="urn:adsk.eagle:library:371" deviceset="+3V3" device=""/>
 <part name="GND113" library="supply1" library_urn="urn:adsk.eagle:library:371" deviceset="GND" device=""/>
-<part name="X1" library="con-phoenix-508" library_urn="urn:adsk.eagle:library:176" deviceset="MKDSN1,5/2-5,08" device="" package3d_urn="urn:adsk.eagle:package:9630/1"/>
+<part name="X1" library="con-phoenix-508-jm" deviceset="MKDSN1,5/2-5,08" device="" package3d_urn="urn:adsk.eagle:package:9630/1"/>
 <part name="U1" library="TCLT1600" library_urn="urn:adsk.eagle:library:38706839" deviceset="TCLT1600" device="" package3d_urn="urn:adsk.eagle:package:38706842/1">
 <attribute name="LCSC_PART" value="C553998"/>
@@
 <part name="K1" library="relay" library_urn="urn:adsk.eagle:library:339" deviceset="JT1A?-*" device="-PCB" package3d_urn="urn:adsk.eagle:package:24455/1" technology="DC12V" value="T90-12VDC-TL-A"/>
 <part name="K2" library="relay" library_urn="urn:adsk.eagle:library:339" deviceset="JT1A?-*" device="-PCB" package3d_urn="urn:adsk.eagle:package:24455/1" technology="DC12V" value="T90-12VDC-TL-A"/>
-<part name="X3" library="con-phoenix-508" library_urn="urn:adsk.eagle:library:176" deviceset="MKDSN1,5/5-5,08" device="" package3d_urn="urn:adsk.eagle:package:9639/1"/>
+<part name="X3" library="con-phoenix-508-jm" deviceset="MKDSN1,5/5-5,08" device="" package3d_urn="urn:adsk.eagle:package:9639/1"/>
 <part name="C9" library="JLC PCB Basic Parts_loc" library_urn="urn:adsk.eagle:library:38668506" deviceset="C_" device="_1206" package3d_urn="urn:adsk.eagle:package:23618/2" technology="100UF/6.3V"/>
 <part name="C10" library="JLC PCB Basic Parts_loc" library_urn="urn:adsk.eagle:library:38668506" deviceset="C_" device="_1206" package3d_urn="urn:adsk.eagle:package:23618/2" technology="100UF/6.3V"/>
@@
 <part name="R56" library="varistor" library_urn="urn:adsk.eagle:library:410" deviceset="S14K420" device="" package3d_urn="urn:adsk.eagle:package:30565/1"/>
 <part name="R57" library="varistor" library_urn="urn:adsk.eagle:library:410" deviceset="S14K420" device="" package3d_urn="urn:adsk.eagle:package:30565/1"/>
-<part name="FIRE" library="con-phoenix-508" library_urn="urn:adsk.eagle:library:176" deviceset="MKDSN1,5/8-5,08" device="" package3d_urn="urn:adsk.eagle:package:9632/1"/>
+<part name="FIRE" library="con-phoenix-508-jm" deviceset="MKDSN1,5/8-5,08" device="" package3d_urn="urn:adsk.eagle:package:9632/1"/>
 <part name="R26" library="JLC PCB Basic Parts_loc" library_urn="urn:adsk.eagle:library:38668506" deviceset="R_" device="_0603" package3d_urn="urn:adsk.eagle:package:23555/3" technology="3K"/>
 <part name="R27" library="JLC PCB Basic Parts_loc" library_urn="urn:adsk.eagle:library:38668506" deviceset="R_" device="_0603" package3d_urn="urn:adsk.eagle:package:23555/3" technology="3K"/>
@@
 <part name="GND28" library="supply1" library_urn="urn:adsk.eagle:library:371" deviceset="GND" device=""/>
 <part name="C32" library="JLC PCB Basic Parts_loc" library_urn="urn:adsk.eagle:library:38668506" deviceset="C_" device="_0603" package3d_urn="urn:adsk.eagle:package:38668554/1" technology="1UF/50V"/>
-<part name="5V_CTRL_LAZERS" library="con-jst-ph" library_urn="urn:adsk.eagle:library:37597460" deviceset="B8B-PH-K" device="" package3d_urn="urn:adsk.eagle:package:37597503/1"/>
+<part name="5V_CTRL_LAZERS" library="con-jst-ph" library_urn="urn:adsk.eagle:library:37597460" deviceset="B8B-PH-K" device="" package3d_urn="urn:adsk.eagle:package:37597503/2"/>
 <part name="P+4" library="supply1" library_urn="urn:adsk.eagle:library:371" deviceset="+5V" device=""/>
 <part name="D2" library="SparkFun-LED" library_urn="urn:adsk.eagle:library:529" deviceset="LED" device="0603" package3d_urn="urn:adsk.eagle:package:39354/1" value="blue">
@@
 <part name="JP2" library="pinhead" library_urn="urn:adsk.eagle:library:325" deviceset="PINHD-2X2" device="" package3d_urn="urn:adsk.eagle:package:22455/2"/>
 <part name="GND32" library="supply1" library_urn="urn:adsk.eagle:library:371" deviceset="GND" device=""/>
+<part name="R6" library="JLC PCB Basic Parts_loc" library_urn="urn:adsk.eagle:library:38668506" deviceset="R_" device="_1206" package3d_urn="urn:adsk.eagle:package:23540/2" technology="0R"/>
+<part name="GND33" library="supply1" library_urn="urn:adsk.eagle:library:371" deviceset="GND" device=""/>
+<part name="SUPPLY14" library="supply2" library_urn="urn:adsk.eagle:library:372" deviceset="GND2" device=""/>
 </parts>
 <sheets>
@@
 <attribute name="VALUE" x="226.06" y="391.16" size="1.778" layer="96"/>
 </instance>
+<instance part="R6" gate="R1" x="406.4" y="396.24" smashed="yes">
+<attribute name="NAME" x="402.59" y="397.7386" size="1.778" layer="95"/>
+<attribute name="VALUE" x="402.59" y="392.938" size="1.778" layer="96"/>
+</instance>
+<instance part="GND33" gate="1" x="398.78" y="391.16" smashed="yes">
+<attribute name="VALUE" x="396.24" y="388.62" size="1.778" layer="96"/>
+</instance>
+<instance part="SUPPLY14" gate="G$1" x="414.02" y="391.16" smashed="yes">
+<attribute name="VALUE" x="411.607" y="387.985" size="1.778" layer="96"/>
+</instance>
 </instances>
 <busses>
@@
 <junction x="238.76" y="401.32"/>
 </segment>
+<segment>
+<pinref part="R6" gate="R1" pin="1"/>
+<pinref part="GND33" gate="1" pin="GND"/>
+<wire x1="401.32" y1="396.24" x2="398.78" y2="396.24" width="0.1524" layer="91"/>
+<wire x1="398.78" y1="396.24" x2="398.78" y2="393.7" width="0.1524" layer="91"/>
+</segment>
 </net>
 <net name="N$1" class="0">
@@
 <wire x1="160.02" y1="116.84" x2="160.02" y2="111.76" width="0.1524" layer="91"/>
 </segment>
+<segment>
+<pinref part="R6" gate="R1" pin="2"/>
+<wire x1="411.48" y1="396.24" x2="414.02" y2="396.24" width="0.1524" layer="91"/>
+<wire x1="414.02" y1="396.24" x2="414.02" y2="393.7" width="0.1524" layer="91"/>
+<pinref part="SUPPLY14" gate="G$1" pin="GND2"/>
+</segment>
 </net>

Commit message: Added buckboost
Parts:
- removed C26, C30: 1uf, rcl:C-USC0805
- removed C27, C31: 10uf, rcl:C-USC0603
- removed C29: (no value), rcl:CPOL-USE10-25
- removed D10, D11: MBR20200CT, MBR20200CT:MBR20200CT
- removed IC5, IC6, IC7: LM317MABDT, v-reg:LM317MABDT
- removed R50, R53, R58: R_240R_0603, JLC PCB Basic Parts_loc:R_240R_0603
- removed R51, R54, R59: R_750R_0603, JLC PCB Basic Parts_loc:R_750R_0603
- removed R52, R6: R_0R_1206, JLC PCB Basic Parts_loc:R_0R_1206
- removed R57: S14K420, varistor:S14K420
- added K5, K6: AQG22110, relay:AQG22110
- added U$2: ZK-SJVA-4X, Nova:ZK-SJVA-4X
- added X2: MKDSN1,5/2-5,08, con-phoenix-508-jm:MKDSN1,5/2-5,08
- C25: value 10uf -> 1uf; device rcl:C-USC0603 -> rcl:C-USC0805; LCSC_PART C19702 -> C15849
- R55, R56: value S14K420 -> S10K40; device varistor:S14K420 -> varistor:S10K40
- R60, R61: value R_56K_0805 -> R_1K_0603; device JLC PCB Basic Parts_loc:R_56K_0805 -> JLC PCB Basic Parts_loc:R_1K_0603
- R62: value R_56K_0805 -> R_7.5K_0603; device JLC PCB Basic Parts_loc:R_56K_0805 -> JLC PCB Basic Parts_loc:R_7.5K_0603
- R63: value R_2.2K_0603 -> R_1K_0603; device JLC PCB Basic Parts_loc:R_2.2K_0603 -> JLC PCB Basic Parts_loc:R_1K_0603
Connections:
- removed net +6V: D15.C, D16.A, FIRE-1.KL, IC5.OUT, IC6.OUT, IC7.OUT, R50.2, R53.2, R58.2
- removed net 60VDC: C29.+, D10.C, D12.C, D13.C, D14.C, D17.A, D18.A, D19.A, FIRE-3.KL, FIRE-5.KL, FIRE-7.KL
- removed net N$53: IC7.ADJ, R58.1, R59.2
- new net +14V: C25.1, D14.C, D17.A, FIRE-3.KL, U$2.OUT+
- new net +5V/2: D15.C, D16.A, FIRE-1.KL, X2-2.KL
- net +12V: now also U$2.IN+; no longer C25.1, C26.1, C27.1, C30.1, C31.1, IC5.IN, IC6.IN, IC7.IN
- net +5V: now also D12.C, D13.C, D18.A, D19.A, K5.A, K6.A
- net 120_LINE: now also K5.DS2, K6.DS2; no longer D10.A1, D10.A2, R57.1
- net 120_NEUTRAL: now also FIRE-6.KL, FIRE-8.KL; no longer D11.C, R57.2
- net GND: now also C24.2, C25.2, Q3.S, U$2.IN-, U$2.OUT-, X2-1.KL; no longer R52.1, R6.1
- net GND2: no longer C29.-, D11.A1, D11.A2, Q3.S, R6.2
- net GND3: no longer C24.2, C25.2, C26.2, C27.2, C30.2, C31.2, R51.1, R52.2, R54.1, R59.1
- net N$47: now also K5.K; no longer FIRE-6.KL
- net N$48: now also FIRE-7.KL, K6.DS1; no longer IC6.ADJ, R53.1, R54.2
- net N$49: now also K6.K; no longer FIRE-8.KL
- net N$50: now also FIRE-5.KL, K5.DS1; no longer IC5.ADJ, R50.1, R51.2
Other:
- moved on the sheet: C24, C25, D14, D15, D16, D17, FIRE-1, FIRE-2, FIRE-3, FIRE-4, FIRE-5, FIRE-6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
