File: hardware/star/star.sch (EAGLE design)
At the start: 151 parts, among them IC1 MAX481CSA, IC2 LD117AS12TR, IC22 LD117AS12TR, IC3 74HCT08D, IC4 7404D, IC8 MAX481CSA, IC9 LD117AS12TR, K1 T90-12VDC-TL-A, K2 T90-12VDC-TL-A, K5 AQG22110, K6 AQG22110, P1 B3B-PH-K, Q1 35A/25V/8.5mΩ, Q2 35A/25V/8.5mΩ, Q3 35A/25V/8.5mΩ, Q4 35A/25V/8.5mΩ, T1 T_PNP_MMBT5401_CHANGJ_SOT23-B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, T2 T_PNP_MMBT5401_CHANGJ_SOT23-B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, T3 T_PNP_MMBT5401_CHANGJ_SOT23-B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, T4 T_PNP_MMBT5401_CHANGJ_SOT23-B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, U1 TCLT1600, X1 MKDSN1,5/2-5,08, X2 MKDSN1,5/2-5,08, X3 MKDSN1,5/5-5,08

Commit message: Add TVS diodes
Parts:
- removed C34: 1uf, rcl:C-USC0805
- removed C37: 10uf, rcl:C-USC0603
- removed IC9: LD117AS12TR, v-reg:LD117AS12TR
- added D4, TVS1, TVS2, TVS3, TVS4: (no value), diode:DIODE-DO214AA
- R14, R23, R32, R39: value R_2K_0603 -> R_10K_0603; device JLC PCB Basic Parts_loc:R_2K_0603 -> JLC PCB Basic Parts_loc:R_10K_0603
- R22, R31, R38, R9: value R_7.5K_0603 -> R_330R_0603; device JLC PCB Basic Parts_loc:R_7.5K_0603 -> JLC PCB Basic Parts_loc:R_330R_0603
- R55, R56: value S10K40 -> S20K20; device varistor:S10K40 -> varistor:S20K20
Connections:
- net +12V: no longer C34.1, IC9.IN, R14.2, R23.2, R32.2, R39.2
- net +5V: no longer C37.1, IC9.OUT
- net GND: now also D4.A, R14.1, R23.1, R32.1, R39.1, TVS1.A, TVS2.A, TVS3.A, TVS4.A; no longer C34.2, C37.2, IC9.ADJ
- net N$17: now also R14.2, TVS1.C; no longer R14.1
- net N$23: now also D4.C
- net N$25: now also R23.2, TVS4.C; no longer R23.1
- net N$31: now also R32.2, TVS2.C; no longer R32.1
- net N$37: now also R39.2, TVS3.C; no longer R39.1
Other:
- note added: "Todo: Drive Q4 with +5 and GND Add Relay to switch +5/2 and GND3"
- moved on the sheet: C15, C19, C21, C23, R14, R22, R23, R31, R32, R38, R39, R9
