File: hardware/star/star.sch (EAGLE design)
At the start: 160 parts, among them IC1 MAX481CSA, IC2 74HCT08D, IC22 LD117AS12TR, IC3 74HCT08D, IC4 7404D, IC8 MAX481CSA, K1 T90-12VDC-TL-A, K2 T90-12VDC-TL-A, K3 T90-12VDC-TL-A, K5 AQG22110, K6 AQG22110, Q1 35A/25V/8.5mΩ, Q2 35A/25V/8.5mΩ, Q3 35A/25V/8.5mΩ, Q4 35A/25V/8.5mΩ, U1 TCLT1600, U2 ADXL343BCCZ-RL7, U3 TMP102AIDRLR, U4 SN74LVC1G17DCK, U5 SN74LVC1G17DCK, U6 SN74LVC1G17DCK, U7 SN74LVC1G17DCK, X1 MKDSN1,5/2-5,08

Commit message: Initial code for starbase
Parts:
- removed R63: R_1K_0603, JLC PCB Basic Parts_loc:R_1K_0603
- added R15: R_2K_0603, JLC PCB Basic Parts_loc:R_2K_0603
Connections:
- net +12V: now also D15.C, D16.A, K3G$1.1
- net +5V: no longer D15.C, D16.A, K3G$1.1
- net N$52: now also R15.2; no longer R63.2
- net N$54: now also R15.1; no longer R63.1
Changed lines of the file:
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@@
 <part name="R61" library="JLC PCB Basic Parts_loc" library_urn="urn:adsk.eagle:library:38668506" deviceset="R_" device="_0603" package3d_urn="urn:adsk.eagle:package:23555/3" technology="1K" value="R_1K_0603"/>
 <part name="R62" library="JLC PCB Basic Parts_loc" library_urn="urn:adsk.eagle:library:38668506" deviceset="R_" device="_0603" package3d_urn="urn:adsk.eagle:package:23555/3" technology="15K" value="R_15K_0603"/>
-<part name="R63" library="JLC PCB Basic Parts_loc" library_urn="urn:adsk.eagle:library:38668506" deviceset="R_" device="_0603" package3d_urn="urn:adsk.eagle:package:23555/3" technology="1K" value="R_1K_0603"/>
 <part name="P+24" library="supply1" library_urn="urn:adsk.eagle:library:371" deviceset="+5V" device=""/>
 <part name="GND28" library="supply1" library_urn="urn:adsk.eagle:library:371" deviceset="GND" device=""/>
@@
 <part name="GND31" library="supply1" library_urn="urn:adsk.eagle:library:371" deviceset="GND" device=""/>
 <part name="SUPPLY6" library="supply2" library_urn="urn:adsk.eagle:library:372" deviceset="+5V/2" device=""/>
-<part name="P+3" library="supply1" library_urn="urn:adsk.eagle:library:371" deviceset="+5V" device=""/>
 <part name="K3" library="relay" library_urn="urn:adsk.eagle:library:339" deviceset="JT1A?-*" device="-PCB" package3d_urn="urn:adsk.eagle:package:24455/1" technology="DC12V" value="T90-12VDC-TL-A"/>
 <part name="LED_ARRAY" library="con-jst-ph" library_urn="urn:adsk.eagle:library:37597460" deviceset="B4B-PH-K" device="" package3d_urn="urn:adsk.eagle:package:37597507/2"/>
@@
 <part name="GND60" library="supply1" library_urn="urn:adsk.eagle:library:371" deviceset="GND" device=""/>
 <part name="+3V23" library="supply1" library_urn="urn:adsk.eagle:library:371" deviceset="+3V3" device=""/>
+<part name="P+3" library="supply1" library_urn="urn:adsk.eagle:library:371" deviceset="+12V" device=""/>
+<part name="R15" library="JLC PCB Basic Parts_loc" library_urn="urn:adsk.eagle:library:38668506" deviceset="R_" device="_0603" package3d_urn="urn:adsk.eagle:package:23555/3" technology="2K"/>
 </parts>
 <sheets>
@@
 <attribute name="VALUE" x="184.15" y="105.918" size="1.778" layer="96"/>
 </instance>
-<instance part="R63" gate="R1" x="170.18" y="38.1" smashed="yes">
-<attribute name="NAME" x="166.37" y="39.5986" size="1.778" layer="95"/>
-<attribute name="VALUE" x="166.37" y="34.798" size="1.778" layer="96"/>
-</instance>
 <instance part="P+24" gate="1" x="274.32" y="261.62" smashed="yes">
 <attribute name="VALUE" x="271.78" y="256.54" size="1.778" layer="96" rot="R90"/>
@@
 <attribute name="VALUE" x="207.01" y="59.055" size="1.778" layer="96"/>
 </instance>
-<instance part="P+3" gate="1" x="172.72" y="58.42" smashed="yes">
-<attribute name="VALUE" x="170.18" y="53.34" size="1.778" layer="96" rot="R90"/>
-</instance>
 <instance part="K3" gate="G$1" x="190.5" y="45.72" smashed="yes">
 <attribute name="VALUE" x="191.77" y="48.641" size="1.778" layer="96"/>
@@
 <attribute name="VALUE" x="93.98" y="53.34" size="1.778" layer="96" rot="R90"/>
 </instance>
+<instance part="P+3" gate="1" x="172.72" y="60.96" smashed="yes">
+<attribute name="VALUE" x="170.18" y="55.88" size="1.778" layer="96" rot="R90"/>
+</instance>
+<instance part="R15" gate="R1" x="170.18" y="38.1" smashed="yes">
+<attribute name="NAME" x="166.37" y="39.5986" size="1.778" layer="95"/>
+<attribute name="VALUE" x="166.37" y="34.798" size="1.778" layer="96"/>
+</instance>
 </instances>
 <busses>
@@
 <junction x="416.56" y="411.48"/>
 </segment>
+<segment>
+<pinref part="D15" gate="D1" pin="C"/>
+<wire x1="177.8" y1="48.26" x2="177.8" y2="53.34" width="0.1524" layer="91"/>
+<junction x="177.8" y="53.34"/>
+<pinref part="D16" gate="G$1" pin="A"/>
+<wire x1="177.8" y1="53.34" x2="172.72" y2="53.34" width="0.1524" layer="91"/>
+<wire x1="172.72" y1="53.34" x2="162.56" y2="53.34" width="0.1524" layer="91"/>
+<wire x1="162.56" y1="53.34" x2="162.56" y2="48.26" width="0.1524" layer="91"/>
+<wire x1="190.5" y1="53.34" x2="177.8" y2="53.34" width="0.1524" layer="91"/>
+<pinref part="K3" gate="G$1" pin="1"/>
+<wire x1="190.5" y1="50.8" x2="190.5" y2="53.34" width="0.1524" layer="91"/>
+<pinref part="P+3" gate="1" pin="+12V"/>
+<wire x1="172.72" y1="58.42" x2="172.72" y2="53.34" width="0.1524" layer="91"/>
+<junction x="172.72" y="53.34"/>
+</segment>
 </net>
 <net name="+5V" class="3">
@@
 </segment>
 <segment>
-<pinref part="D15" gate="D1" pin="C"/>
-<wire x1="177.8" y1="48.26" x2="177.8" y2="53.34" width="0.1524" layer="91"/>
-<junction x="177.8" y="53.34"/>
-<pinref part="D16" gate="G$1" pin="A"/>
-<wire x1="177.8" y1="53.34" x2="172.72" y2="53.34" width="0.1524" layer="91"/>
-<wire x1="172.72" y1="53.34" x2="162.56" y2="53.34" width="0.1524" layer="91"/>
-<wire x1="162.56" y1="53.34" x2="162.56" y2="48.26" width="0.1524" layer="91"/>
-<pinref part="P+3" gate="1" pin="+5V"/>
-<wire x1="172.72" y1="53.34" x2="172.72" y2="55.88" width="0.1524" layer="91"/>
-<junction x="172.72" y="53.34"/>
-<wire x1="190.5" y1="53.34" x2="177.8" y2="53.34" width="0.1524" layer="91"/>
-<pinref part="K3" gate="G$1" pin="1"/>
-<wire x1="190.5" y1="50.8" x2="190.5" y2="53.34" width="0.1524" layer="91"/>
-</segment>
-<segment>
 <pinref part="P+21" gate="1" pin="+5V"/>
 <pinref part="NID35-5" gate="G$1" pin="OUT4"/>
@@
 <pinref part="K3" gate="G$1" pin="2"/>
 <wire x1="190.5" y1="38.1" x2="190.5" y2="40.64" width="0.1524" layer="91"/>
-<pinref part="R63" gate="R1" pin="2"/>
 <wire x1="175.26" y1="38.1" x2="177.8" y2="38.1" width="0.1524" layer="91"/>
 <junction x="177.8" y="38.1"/>
+<pinref part="R15" gate="R1" pin="2"/>
 </segment>
 </net>
@@
 <pinref part="D16" gate="G$1" pin="C"/>
 <wire x1="162.56" y1="40.64" x2="162.56" y2="38.1" width="0.1524" layer="91"/>
-<pinref part="R63" gate="R1" pin="1"/>
 <wire x1="162.56" y1="38.1" x2="165.1" y2="38.1" width="0.1524" layer="91"/>
+<pinref part="R15" gate="R1" pin="1"/>
 </segment>
 </net>
